File: Filters.sch (KiCad schematic (older format))
At the start: 18 parts

Commit message: Updated PCB layout to reflect changes in footprints.
Parts:
- C401, C402, C403, C404, C405, C406: footprint Newlib:CAPRR_P100W40L125 -> Newlib:CAPRR_P50W25L72
Changed lines of the file:
@@
 EESchema Schematic File Version 2
-LIBS:z_newlib
-LIBS:z_power
 LIBS:stereo_amp-cache
-EELAYER 25 0
+EELAYER 24 0
 EELAYER END
 $Descr A4 11693 8268
@@
 F 0 "C401" H 4275 3825 50  0000 L BNN
 F 1 "15n" H 4275 3775 50  0000 L TNN
-F 2 "Newlib:CAPRR_P100W40L125" H 4250 3800 60  0001 C CNN
+F 2 "Newlib:CAPRR_P50W25L72" H 4250 3800 60  0001 C CNN
 F 3 "" H 4250 3800 60  0000 C CNN
 	1    4250 3800
@@
 F 0 "C403" H 4525 4425 50  0000 L BNN
 F 1 "10n" V 4550 4250 50  0000 L TNN
-F 2 "Newlib:CAPRR_P100W40L125" H 4500 4400 60  0001 C CNN
+F 2 "Newlib:CAPRR_P50W25L72" H 4500 4400 60  0001 C CNN
 F 3 "" H 4500 4400 60  0000 C CNN
 	1    4500 4400
@@
 F 0 "C405" H 5075 4175 50  0000 L BNN
 F 1 "15n" V 5100 4000 50  0000 L TNN
-F 2 "Newlib:CAPRR_P100W40L125" H 5050 4150 60  0001 C CNN
+F 2 "Newlib:CAPRR_P50W25L72" H 5050 4150 60  0001 C CNN
 F 3 "" H 5050 4150 60  0000 C CNN
 	1    5050 4150
@@
 F 0 "C404" H 4525 5625 50  0000 L BNN
 F 1 "10n" V 4550 5450 50  0000 L TNN
-F 2 "Newlib:CAPRR_P100W40L125" H 4500 5600 60  0001 C CNN
+F 2 "Newlib:CAPRR_P50W25L72" H 4500 5600 60  0001 C CNN
 F 3 "" H 4500 5600 60  0000 C CNN
 	1    4500 5600
@@
 F 0 "C402" H 4275 6225 50  0000 L BNN
 F 1 "15n" H 4275 6175 50  0000 L TNN
-F 2 "Newlib:CAPRR_P100W40L125" H 4250 6200 60  0001 C CNN
+F 2 "Newlib:CAPRR_P50W25L72" H 4250 6200 60  0001 C CNN
 F 3 "" H 4250 6200 60  0000 C CNN
 	1    4250 6200
@@
 F 0 "C406" H 5075 5875 50  0000 L BNN
 F 1 "15n" V 5100 5700 50  0000 L TNN
-F 2 "Newlib:CAPRR_P100W40L125" H 5050 5850 60  0001 C CNN
+F 2 "Newlib:CAPRR_P50W25L72" H 5050 5850 60  0001 C CNN
 F 3 "" H 5050 5850 60  0000 C CNN
 	1    5050 5850
