File: supply.sch (KiCad schematic (older format))
At the start: 4 parts

Commit message: Finished placement and routing.
Changed lines of the file:
@@
 AR Path="/543EAC44/543F2EEA" Ref="D501"  Part="1"
 AR Path="/543ED58C/543F2EEA" Ref="D601"  Part="1"
-F 0 "D501" H 3700 3300 60  0000 C CNN
+F 0 "D601" H 3700 3300 60  0000 C CNN
 F 1 "BRIDGERECT" H 3900 2900 60  0000 C CNN
 F 2 "Newlib:KBPC606" H 3550 3100 60  0001 C CNN
@@
 	3900 3100 3800 3100
 $Comp
-L GND #PWR028
+L GND #PWR501
 U 1 1 543F2F62
 P 4500 3750
-AR Path="/543EAC44/543F2F62" Ref="#PWR028"  Part="1"
-AR Path="/543ED58C/543F2F62" Ref="#PWR029"  Part="1"
-F 0 "#PWR029" H 4500 3710 30  0001 C CNN
+AR Path="/543EAC44/543F2F62" Ref="#PWR501"  Part="1"
+AR Path="/543ED58C/543F2F62" Ref="#PWR601"  Part="1"
+F 0 "#PWR601" H 4500 3710 30  0001 C CNN
 F 1 "GND" H 4500 3635 30  0001 C CNN
 F 2 "" H 4500 3750 60  0000 C CNN
@@
 AR Path="/543EAC44/543F2FC9" Ref="C501"  Part="1"
 AR Path="/543ED58C/543F2FC9" Ref="C601"  Part="1"
-F 0 "C501" V 3200 3400 50  0000 L BNN
+F 0 "C601" V 3200 3400 50  0000 L BNN
 F 1 "0.47u" V 3000 3400 50  0000 L TNN
 F 2 "Newlib:CAPRR_P50W60L72" H 3100 3350 60  0001 C CNN
@@
 AR Path="/543EAC44/543F310E" Ref="C502"  Part="1"
 AR Path="/543ED58C/543F310E" Ref="C602"  Part="1"
-F 0 "C502" V 4000 2900 50  0000 L BNN
+F 0 "C602" V 4000 2900 50  0000 L BNN
 F 1 "47n" V 3800 2900 50  0000 L TNN
 F 2 "Newlib:CAPRR_P150W50L180" H 3900 2850 60  0001 C CNN
@@
 AR Path="/543EAC44/543F31B3" Ref="C503"  Part="1"
 AR Path="/543ED58C/543F31B3" Ref="C603"  Part="1"
-F 0 "C503" V 4400 3200 50  0000 L BNN
+F 0 "C603" V 4400 3200 50  0000 L BNN
 F 1 "3300u" V 4450 3250 50  0000 L TNN
 F 2 "Newlib:CAPPR_P75D180" H 4500 3150 60  0001 C CNN

Commit message: Updated PCB layout to reflect changes in footprints.
Parts:
- C501: footprint Newlib:CAPRR_P50W60L72 -> Newlib:CAPRR_P50W50L72
- C502: footprint Newlib:CAPRR_P150W50L180 -> Newlib:CAPRR_P50W25L72
Changed lines of the file:
@@
 EESchema Schematic File Version 2
-LIBS:z_newlib
-LIBS:z_power
 LIBS:stereo_amp-cache
-EELAYER 25 0
+EELAYER 24 0
 EELAYER END
 $Descr A4 11693 8268
@@
 F 0 "C601" V 3200 3400 50  0000 L BNN
 F 1 "0.47u" V 3000 3400 50  0000 L TNN
-F 2 "Newlib:CAPRR_P50W60L72" H 3100 3350 60  0001 C CNN
+F 2 "Newlib:CAPRR_P50W50L72" H 3100 3350 60  0001 C CNN
 F 3 "" H 3100 3350 60  0000 C CNN
 	1    3100 3350
@@
 F 0 "C602" V 4000 2900 50  0000 L BNN
 F 1 "47n" V 3800 2900 50  0000 L TNN
-F 2 "Newlib:CAPRR_P150W50L180" H 3900 2850 60  0001 C CNN
+F 2 "Newlib:CAPRR_P50W25L72" H 3900 2850 60  0001 C CNN
 F 3 "" H 3900 2850 60  0000 C CNN
 	1    3900 2850
